Commit message: 修改URDF和配置文件

File: src/arm_model/model/robotic_arm.urdf (robot description, URDF)
Before this commit: robot robotic_arm, 8 links, 7 joints
Links:
- link base_link: geometry collision mesh filename=package://arm_model/model/base_link.STL; visual mesh filename=package://arm_model/model/base_link.STL
- link link1: geometry collision mesh filename=package://arm_model/model/link1.STL; visual mesh filename=package://arm_model/model/link1.STL
- link link2: geometry collision mesh filename=package://arm_model/model/link2.STL; visual mesh filename=package://arm_model/model/link2.STL
- link link3: geometry collision mesh filename=package://arm_model/model/link3.STL; visual mesh filename=package://arm_model/model/link3.STL
- link link4: geometry collision mesh filename=package://arm_model/model/link4.STL; visual mesh filename=package://arm_model/model/link4.STL
- link link5: geometry collision mesh filename=package://arm_model/model/link5.STL; visual mesh filename=package://arm_model/model/link5.STL
- link link6: geometry collision mesh filename=package://arm_model/model/link6.STL; visual mesh filename=package://arm_model/model/link6.STL
